Commit message: Remove unnecesary dummy joints/links from URDF.

File: lwr_description/model/kuka_lwr.urdf.xacro (robot description, xacro)
@@ -55,12 +55,4 @@
 			<child link="${name}_1_link"/>
 		</joint>
-		<joint name="${name}_0_joint_stiffness" type="revolute">
-			<axis xyz="0 0 1"/>
-			<limit lower="${min_stiffness}" upper="${max_stiffness}" effort="0" velocity="${rate_stiffness}" />
-			<safety_controller soft_lower_limit="${min_stiffness}" soft_upper_limit="${max_stiffness}" k_position="30" k_velocity="30"/>
-			<parent link="${name}_base_link"/>
-			<child link="${name}_1_link_dummy"/>
-		</joint>
-		<link name="${name}_1_link_dummy"/>
 		<link name="${name}_1_link">
 			<inertial>
@@ -105,12 +97,4 @@
 			<child link="${name}_2_link"/>
 		</joint>
-		<joint name="${name}_1_joint_stiffness" type="revolute">
-			<axis xyz="0 0 1"/>
-			<limit lower="${min_stiffness}" upper="${max_stiffness}" effort="0" velocity="${rate_stiffness}" />
-			<safety_controller soft_lower_limit="${min_stiffness}" soft_upper_limit="${max_stiffness}" k_position="30" k_velocity="30"/>
-			<parent link="${name}_1_link"/>
-			<child link="${name}_2_link_dummy"/>
-		</joint>
-		<link name="${name}_2_link_dummy"/>
 		<link name="${name}_2_link">
 			<inertial>
@@ -155,12 +139,4 @@
 			<child link="${name}_3_link"/>
 		</joint>
-		<joint name="${name}_2_joint_stiffness" type="revolute">
-			<axis xyz="0 0 1"/>
-			<limit lower="${min_stiffness}" upper="${max_stiffness}" effort="0" velocity="${rate_stiffness}" />
-			<safety_controller soft_lower_limit="${min_stiffness}" soft_upper_limit="${max_stiffness}" k_position="30" k_velocity="30"/>
-			<parent link="${name}_2_link"/>
-			<child link="${name}_3_link_dummy"/>
-		</joint>
-		<link name="${name}_3_link_dummy"/>
 		<link name="${name}_3_link">
 			<inertial>
@@ -205,12 +181,4 @@
 			<child link="${name}_4_link"/>
 		</joint>
-		<joint name="${name}_3_joint_stiffness" type="revolute">
-			<axis xyz="0 0 1"/>
-			<limit lower="${min_stiffness}" upper="${max_stiffness}" effort="0" velocity="${rate_stiffness}" />
-			<safety_controller soft_lower_limit="${min_stiffness}" soft_upper_limit="${max_stiffness}" k_position="30" k_velocity="30"/>
-			<parent link="${name}_3_link"/>
-			<child link="${name}_4_link_dummy"/>
-		</joint>
-		<link name="${name}_4_link_dummy"/>
 		<link name="${name}_4_link">
 			<inertial>
@@ -255,12 +223,4 @@
 			<child link="${name}_5_link"/>
 		</joint>
-		<joint name="${name}_4_joint_stiffness" type="revolute">
-			<axis xyz="0 0 1"/>
-			<limit lower="${min_stiffness}" upper="${max_stiffness}" effort="0" velocity="${rate_stiffness}" />
-			<safety_controller soft_lower_limit="${min_stiffness}" soft_upper_limit="${max_stiffness}" k_position="30" k_velocity="30"/>
-			<parent link="${name}_4_link"/>
-			<child link="${name}_5_link_dummy"/>
-		</joint>
-		<link name="${name}_5_link_dummy"/>
 		<link name="${name}_5_link">
 			<inertial>
@@ -305,12 +265,4 @@
 			<child link="${name}_6_link"/>
 		</joint>
-		<joint name="${name}_5_joint_stiffness" type="revolute">
-			<axis xyz="0 0 1"/>
-			<limit lower="${min_stiffness}" upper="${max_stiffness}" effort="0" velocity="${rate_stiffness}" />
-			<safety_controller soft_lower_limit="${min_stiffness}" soft_upper_limit="${max_stiffness}" k_position="30" k_velocity="30"/>
-			<parent link="${name}_5_link"/>
-			<child link="${name}_6_link_dummy"/>
-		</joint>
-		<link name="${name}_6_link_dummy"/>
 		<link name="${name}_6_link">
 			<inertial>
@@ -342,12 +294,4 @@
 			<child link="${name}_7_link"/>
 		</joint>
-		<joint name="${name}_6_joint_stiffness" type="revolute">
-			<axis xyz="0 0 1"/>
-			<limit lower="${min_stiffness}" upper="${max_stiffness}" effort="0" velocity="${rate_stiffness}" />
-			<safety_controller soft_lower_limit="${min_stiffness}" soft_upper_limit="${max_stiffness}" k_position="30" k_velocity="30"/>
-			<parent link="${name}_6_link"/>
-			<child link="${name}_7_link_dummy"/>
-		</joint>
-		<link name="${name}_7_link_dummy"/>
 		<link name="${name}_7_link">
 			<inertial>

Commit message: Add xacro parameters to tune controller period in simulation.

File: lwr_description/model/kuka_lwr.urdf.xacro (robot description, xacro)
@@ -19,5 +19,5 @@
 	<xacro:property name="rate_stiffness" value="20000"/> <!-- reflex to stiffness -->
 	<!-- URDF model /-->
-	<xacro:macro name="kuka_lwr" params="parent name *origin">
+	<xacro:macro name="kuka_lwr" params="parent name gazebo_control_period:=0 *origin">
 		<!-- First (shoulder) element of the arm. Fixed to its parent. -->
 		<joint name="${parent}_${name}_base_joint" type="fixed">
@@ -366,5 +366,5 @@
 			</collision>
 		</link>
-		<xacro:kuka_lwr_gazebo name="${name}"/>
+		<xacro:kuka_lwr_gazebo name="${name}" control_period="${gazebo_control_period}"/>
 		<xacro:kuka_lwr_transmission name="${name}"/>
 	</xacro:macro>
